File: hardware/picoMBC.kicad_sch (KiCad schematic)
At the start: 9 parts, among them J1 Micro_SD_Card, J2 Conn_02x25_Odd_Even, U1 Pico 2, U2 74LS125

Commit message: Multiplex pico bus
- add buffers to multiplex Pico bus to free up some I/O for future use
Parts:
- removed R2, R3, R4: 4k7, Resistor_THT:R_Axial_DIN0204_L3.6mm_D1.6mm_P7.62mm_Horizontal, symbol Device:R_Small_US
- removed U2: 74LS125, Package_SO:SOIC-14_3.9x8.7mm_P1.27mm, symbol 74xx:74LS125
- added J3: DE9_Plug_MountingHoles, Connector_Dsub:DSUB-9_Male_Horizontal_P2.77x2.84mm_EdgePinOffset4.94mm_Housed_MountingHolesOffset7.48mm, symbol Connector:DE9_Plug_MountingHoles
- added J4: Conn_02x05_Odd_Even, Connector_PinHeader_2.54mm:PinHeader_2x05_P2.54mm_Vertical, symbol Connector_Generic:Conn_02x05_Odd_Even
- added J5: Conn_01x06, Connector_PinHeader_2.54mm:PinHeader_1x06_P2.54mm_Vertical, symbol Connector_Generic:Conn_01x06
- added U2, U5: 74LVC125AD,118, Package_SO:SOIC-14_3.9x8.7mm_P1.27mm, symbol 74xx:74LVC125
- added U3, U4: 74LVC245AD,118, Package_SO:SOIC-20W_7.5x12.8mm_P1.27mm, symbol Logic_LevelTranslator:SN74LVC245APW
- J1: value Micro_SD_Card -> MicroSD
Connections:
- net ~{PICO_INT} is gone; now on net ~{BUS_NMI}: JP1.1 (A)
- net +3.3V: now also R1.1, U2.14 (VCC), U3.20 (VCC), U4.1 (DIR), U4.20 (VCC), U5.14 (VCC)
- net +5V: no longer R1.1
- net BUS_A0: now also U4.9 (A8); no longer U1.11 (GPIO8)
- net BUS_A1: now also U4.8 (A7); no longer U1.12 (GPIO9)
- net BUS_A2: now also U4.7 (A6); no longer U1.14 (GPIO10)
- net BUS_A3: now also U4.6 (A5); no longer U1.15 (GPIO11)
- net BUS_A4: now also U4.5 (A4); no longer U1.16 (GPIO12)
- net BUS_A5: now also U4.4 (A3); no longer U1.17 (GPIO13)
- net BUS_A6: now also U4.3 (A2); no longer U1.19 (GPIO14)
- net BUS_A7: now also U4.2 (A1); no longer U1.20 (GPIO15)
- net BUS_CLOCK: now also U5.9
- net BUS_D0: now also U3.9 (A8); no longer U1.1 (GPIO0)
- net BUS_D1: now also U3.8 (A7); no longer U1.2 (GPIO1)
- net BUS_D2: now also U3.7 (A6); no longer U1.4 (GPIO2)
- net BUS_D3: now also U3.6 (A5); no longer U1.5 (GPIO3)
- net BUS_D4: now also U3.5 (A4); no longer U1.6 (GPIO4)
- net BUS_D5: now also U3.4 (A3); no longer U1.7 (GPIO5)
- net BUS_D6: now also U3.3 (A2); no longer U1.9 (GPIO6)
- net BUS_D7: now also U3.2 (A1); no longer U1.10 (GPIO7)
- net GND: now also J3.0 (PAD), U2.10, U2.13, U2.2, U2.4, U2.7 (GND), U3.10 (GND), U4.10 (GND), U5.7 (GND)
- net ~{BUS_INT}: now also JP1.3 (B)
- net ~{BUS_IORQ}: now also U2.12; no longer U1.27 (GPIO21)
- net ~{BUS_M1}: now also U5.2; no longer U1.26 (GPIO20)
- net ~{BUS_RD}: now also U2.9; no longer U1.32 (GPIO27_ADC1)
- net ~{BUS_RESET}: now also U5.12
- net ~{BUS_WR}: now also U2.5; no longer U1.34 (GPIO28_ADC2)
- net ~{PICO-IRQ}: now also R1.2, U2.1; no longer JP1.2 (C), U1.31 (GPIO26_ADC0)
- net GPIO22: now reaches U1.29 (GPIO22)
- net GPIO22: now also J5.4 (Pin_4)
- removed net ~{PICO_NMI}: JP1.3 (B), R1.2
- new net DE9_1: J3.1, J4.1 (Pin_1)
- new net DE9_2: J3.2, J4.2 (Pin_2)
- new net DE9_3: J3.3, J4.3 (Pin_3)
- new net DE9_4: J3.4, J4.4 (Pin_4)
- new net DE9_5: J3.5, J4.5 (Pin_5)
- new net DE9_6: J3.6, J4.6 (Pin_6)
- new net DE9_7: J3.7, J4.7 (Pin_7)
- new net DE9_8: J3.8, J4.8 (Pin_8)
- new net DE9_9: J3.9, J4.9 (Pin_9)
- new net GPIO20: J5.6 (Pin_6), U1.26 (GPIO20)
- new net GPIO21: J5.5 (Pin_5), U1.27 (GPIO21)
- new net GPIO26: J5.3 (Pin_3), U1.31 (GPIO26_ADC0)
- new net GPIO27: J5.2 (Pin_2), U1.32 (GPIO27_ADC1)
- new net GPIO28: J5.1 (Pin_1), U1.34 (GPIO28_ADC2)
- new net PICO_AD0: U1.1 (GPIO0), U3.11 (B8), U4.11 (B8)
- new net PICO_AD1: U1.2 (GPIO1), U3.12 (B7), U4.12 (B7)
- new net PICO_AD2: U1.4 (GPIO2), U3.13 (B6), U4.13 (B6)
- new net PICO_AD3: U1.5 (GPIO3), U3.14 (B5), U4.14 (B5)
- new net PICO_AD4: U1.6 (GPIO4), U3.15 (B4), U4.15 (B4)
- new net PICO_AD5: U1.7 (GPIO5), U3.16 (B3), U4.16 (B3)
- new net PICO_AD6: U1.9 (GPIO6), U3.17 (B2), U4.17 (B2)
- new net PICO_AD7: U1.10 (GPIO7), U3.18 (B1), U4.18 (B1)
- new net PICO_CLOCK: U1.15 (GPIO11), U5.8
- new net ~{AOE}: U1.19 (GPIO14), U4.19 (~{OE})
- new net ~{BUS_IRQ}: JP1.2 (C), U2.3
- new net ~{DOE}: U1.20 (GPIO15), U3.19 (~{OE})
- new net ~{PICO_IORQ}: U1.14 (GPIO10), U2.11
- new net ~{PICO_M1}: U1.16 (GPIO12), U5.3
- new net ~{PICO_RD}: U1.12 (GPIO9), U2.8, U3.1 (DIR)
- new net ~{PICO_RESET}: U1.17 (GPIO13), U5.11
- new net ~{PICO_WR}: U1.11 (GPIO8), U2.6
Other:
- moved on the sheet: JP1, R1

Commit message: add power header & plot gerbers
Parts:
- added J6: Conn_01x06, Connector_PinHeader_2.54mm:PinHeader_1x06_P2.54mm_Vertical, symbol Connector_Generic:Conn_01x06
Connections:
- net +3.3V: now also J6.1 (Pin_1), J6.2 (Pin_2)
- net +5V: now also J6.5 (Pin_5), J6.6 (Pin_6)
- net GND: now also J6.3 (Pin_3), J6.4 (Pin_4)
